Commit message: Initial URDF/xacro files for robotic arm.

File: src/labra_robot_description/urdf/common_properties.xacro (robot description, xacro)
@@ -9,4 +9,10 @@
     <material name="grey">
         <color rgba="0.5 0.5 0.5 1"/>
+    </material>
+    <material name="orange">
+        <color rgba="1.0 0.647 0.0 1.0"/>
+    </material>
+    <material name="yellow">
+        <color rgba="1.0 1.0 0.0 1.0"/>
     </material>
     <xacro:macro name="box_inertia" params="m x y z o_xyz o_rpy">
