Commit message: Final Project - Adding a robotic arm to a mobile base.

File: src/labra_robot_description/urdf/arm.xacro (robot description, xacro)
@@ -6,5 +6,4 @@
     <xacro:property name="cylinder_radius" value="0.02"/>
     <xacro:property name="cylinder_length" value="0.3"/>
-    <link name="base_footprint"/>
     <link name="arm_base_link">
         <visual>
@@ -13,14 +12,14 @@
             </geometry>
             <origin xyz="0 0 ${arm_base_height / 2.0}" rpy="0 0 0" />
-            <material name="blue" />
+            <material name="orange" />
         </visual>
-        <!-- <collision>
+        <collision>
             <geometry>
-                <box size="${base_length} ${base_width} ${base_height}" />
+                <box size="${arm_base_length} ${arm_base_width} ${arm_base_height}" />
             </geometry>
-            <origin xyz="0 0 ${base_height / 2.0}" rpy="0 0 0" />
+            <origin xyz="0 0 ${arm_base_height / 2.0}" rpy="0 0 0" />
         </collision>
-        <xacro:box_inertia m="5.0" x="${base_length}" y="${base_width}" z="${base_height}"
-                           o_xyz="0 0 ${base_height / 2.0}" o_rpy="0 0 0" /> -->
+        <xacro:box_inertia m="0.5" x="${arm_base_length}" y="${arm_base_width}" z="${arm_base_height}"
+                           o_xyz="0 0 ${arm_base_height / 2.0}" o_rpy="0 0 0" />
     </link>
     <link name="forearm_link">
@@ -30,14 +29,14 @@
             </geometry>
             <origin xyz="0 0 ${cylinder_length/2.0}" rpy="0 0 0" />
-            <material name="blue" />
+            <material name="yellow" />
         </visual>
-        <!-- <collision>
+        <collision>
             <geometry>
-                <box size="${base_length} ${base_width} ${base_height}" />
+                <cylinder radius="${cylinder_radius}" length="${cylinder_length}" />
             </geometry>
-            <origin xyz="0 0 ${base_height / 2.0}" rpy="0 0 0" />
+            <origin xyz="0 0 ${cylinder_length/2.0}" rpy="0 0 0" />
         </collision>
-        <xacro:box_inertia m="5.0" x="${base_length}" y="${base_width}" z="${base_height}"
-                           o_xyz="0 0 ${base_height / 2.0}" o_rpy="0 0 0" /> -->
+        <xacro:cylinder_inertia m="0.3" r="${cylinder_radius}" h="${cylinder_length}"
+                           o_xyz="0 0 ${cylinder_length / 2.0}" o_rpy="0 0 0" />
     </link>
     <link name="hand_link">
@@ -47,19 +46,19 @@
             </geometry>
             <origin xyz="0 0 ${cylinder_length/2.0}" rpy="0 0 0" />
-            <material name="blue" />
+            <material name="orange" />
         </visual>
-        <!-- <collision>
+        <collision>
             <geometry>
-                <box size="${base_length} ${base_width} ${base_height}" />
+                <cylinder radius="${cylinder_radius}" length="${cylinder_length}" />
             </geometry>
-            <origin xyz="0 0 ${base_height / 2.0}" rpy="0 0 0" />
+            <origin xyz="0 0 ${cylinder_length/2.0}" rpy="0 0 0" />
         </collision>
-        <xacro:box_inertia m="5.0" x="${base_length}" y="${base_width}" z="${base_height}"
-                           o_xyz="0 0 ${base_height / 2.0}" o_rpy="0 0 0" /> -->
+        <xacro:cylinder_inertia m="0.3" r="${cylinder_radius}" h="${cylinder_length}"
+                           o_xyz="0 0 ${cylinder_length / 2.0}" o_rpy="0 0 0" />
     </link>
-    <joint name="base_joint" type="fixed">
-        <parent link="base_footprint" />
+    <joint name="base_armbase_joint" type="fixed">
+        <parent link="base_link" />
         <child link="arm_base_link" />
-        <origin xyz="0 0 0" rpy="0 0 0" />
+        <origin xyz="${base_length/4} 0 ${base_height}" rpy="0 0 0" />
     </joint>
     <joint name="base_forearm_joint" type="revolute">
@@ -77,20 +76,3 @@
         <limit effort="1000.0" lower="${-pi/3}" upper="${pi/3}" velocity="0.1"/>
     </joint>
-    <!-- <joint name="base_right_wheel_joint" type="continuous">
-        <parent link="base_link" />
-        <child link="right_wheel_link" />
-        <origin xyz="${-base_length / 4.0} ${-(base_width + wheel_length) / 2.0} 0" rpy="0 0 0" />
-        <axis xyz="0 1 0"/>
-    </joint>
-    <joint name="base_left_wheel_joint" type="continuous">
-        <parent link="base_link" />
-        <child link="left_wheel_link" />
-        <origin xyz="${-base_length / 4.0} ${(base_width + wheel_length) / 2.0} 0" rpy="0 0 0" />
-        <axis xyz="0 1 0"/>
-    </joint>
-    <joint name="base_caster_wheel_joint" type="fixed">
-        <parent link="base_link" />
-        <child link="caster_wheel_link" />
-        <origin xyz="${base_length / 3.0} 0 ${-wheel_radius / 2.0}" rpy="0 0 0" />
-    </joint> -->
 </robot>

File: src/labra_robot_description/urdf/arm_gazebo.xacro (robot description, xacro)
@@ -7,30 +7,8 @@
     <gazebo>
     <plugin
-        filename="gz-sim-diff-drive-system"
-        name="gz::sim::systems::DiffDrive">
-        <left_joint>base_left_wheel_joint</left_joint>
-        <right_joint>base_right_wheel_joint</right_joint>
-        <wheel_separation>0.45</wheel_separation>
-        <wheel_radius>0.1</wheel_radius>
-        <frame_id>odom</frame_id>
-        <child_frame_id>base_footprint</child_frame_id>
-    </plugin>
-    </gazebo>
-    <gazebo>
-    <plugin
         filename="gz-sim-joint-state-publisher-system"
         name="gz::sim::systems::JointStatePublisher">
-        <joint_name>base_left_wheel_joint</joint_name>
-        <joint_name>base_right_wheel_joint</joint_name>
-        <!-- <joint_name>base_forearm_joint</joint_name>
-        <joint_name>forearm_hand_joint</joint_name> -->
-    </plugin>
-    </gazebo>
-    <!-- <gazebo>
-    <plugin
-        filename="gz-sim-joint-position-controller-system"
-        name="gz::sim::systems::JointPositionController">
         <joint_name>base_forearm_joint</joint_name>
-        <p_gain>5.0</p_gain>
+        <joint_name>forearm_hand_joint</joint_name>
     </plugin>
     </gazebo>
@@ -41,5 +19,5 @@
         <joint_name>base_forearm_joint</joint_name>
         <p_gain>5.0</p_gain>
-        <i_gain>1.0</i_gain>
+        <!-- <i_gain>1.0</i_gain> -->
     </plugin>
     </gazebo>
@@ -51,4 +29,4 @@
         <p_gain>3.0</p_gain>
     </plugin>
-    </gazebo> -->
+    </gazebo>
 </robot>

File: src/labra_robot_description/urdf/labra_robot.urdf.xacro (robot description, xacro)
@@ -3,5 +3,7 @@
     <xacro:include filename="common_properties.xacro"/>
     <xacro:include filename="mobile_base.xacro"/>
+    <xacro:include filename="arm.xacro"/>
     <xacro:include filename="mobile_base_gazebo.xacro"/>
+    <xacro:include filename="arm_gazebo.xacro"/>
     <xacro:include filename="camera.xacro"/>
 </robot>

File: src/labra_robot_description/urdf/standalone_arm.urdf.xacro (robot description, xacro)
@@ -3,3 +3,4 @@
     <xacro:include filename="common_properties.xacro"/>
     <xacro:include filename="arm.xacro"/>
+    <xacro:include filename="standalone_arm_gazebo.xacro"/>
 </robot>
